Commit message: Add files via upload

File: m2wr_ws/src/m2wr_description/urdf/m2wr.xacro (robot description, xacro)
@@ -1,50 +1,7 @@
 <?xml version="1.0" ?>
 <robot name="m2wr" xmlns:xacro="http://www.ros.org/wiki/xacro">
-	<material name="black">
-		<color rgba="0.0 0.0 0.0 1.0"/>
-	</material>
-	<material name="blue">
-		<color rgba="0.203125 0.238281250 0.285156250 1.0"/>
-	</material>
-	<material name="green">
-		<color rgba="0.0 0.8 0.0 1.0"/>
-	</material>
-	<material name="grey">
-		<color rgba="0.2 0.2 0.2 1.0"/>
-	</material>
-	<material name="orange">
-		<color rgba="1.0 0.4235294117650 0.0392156862745 1.0"/>
-	</material>
-	<material name="brown">
-		<color rgba="0.870588235294 0.8117647058820 0.7647058823530 1.0"/>
-	</material>
-	<material name="white">
-		<color rgba="1.0 1.0 1.0 1.0"/>
-	</material>
-	<gazebo reference="link_chassis">
-		<material>Gazebo/Orange</material>
-	</gazebo>
-	<gazebo reference="link_right_wheel">
-		<material>Gazebo/Blue</material>
-	</gazebo>
-	<gazebo reference="link_left_wheel">
-		<material>Gazebo/Blue</material>
-	</gazebo>
-	<gazebo>
-		<plugin filename="libgazebo_ros_diff_drive.so" name="differential_drive_controller">
-			<legacyMode>false</legacyMode>
-			<alwaysOn>true</alwaysOn>
-			<updateRate>20</updateRate>
-			<leftJoint>joint_left_wheel</leftJoint>
-			<rightJoint>joint_right_wheel</rightJoint>
-			<wheelSeparation>0.3</wheelSeparation>
-			<wheelDiameter>0.2</wheelDiameter>
-			<torque>0.1</torque>
-			<commandTopic>cmd_vel</commandTopic>
-			<odometryTopic>odom</odometryTopic>
-			<odometryFrame>odom</odometryFrame>
-			<robotBaseFrame>link_chassis</robotBaseFrame>
-		</plugin>
-	</gazebo>
+	<xacro:include filename="$(find m2wr_description)/urdf/materials.xacro" />
+	<xacro:include filename="$(find m2wr_description)/urdf/m2wr.gazebo" />
+	<xacro:include filename="$(find m2wr_description)/urdf/macros.xacro" />
 	<link name="link_chassis">
 		<pose>0 0 0.1 0 0 0</pose>
@@ -89,57 +46,7 @@
 		</visual>
 	</link>
-	<link name="link_right_wheel">
-		<inertial>
-			<mass value="0.2" />
-			<origin rpy="0 1.5707 1.5707" xyz="0 0 0" />
-			<inertia ixx="0.00052666666667" ixy="0" ixz="0" iyy="0.00526666666667" iyz="0" izz="0" />
-		</inertial>
-		<collision name="link_right_wheel_collision">
-			<origin rpy="0 1.5707 1.5707" xyz="0 0 0" />
-			<geometry>
-				<cylinder length="0.04" radius="0.1" />
-			</geometry>
-		</collision>
-		<visual name="link_right_wheel_visual">
-			<origin rpy="0 1.5707 1.5707" xyz="0 0 0" />
-			<geometry>
-				<cylinder length="0.04" radius="0.1" />
-			</geometry>
-		</visual>
-	</link>
-	<link name="link_left_wheel">
-		<inertial>
-			<mass value="0.2" />
-			<origin rpy="0 1.5707 1.5707" xyz="0 0 0" />
-			<inertia ixx="0.00052666666667" ixy="0" ixz="0" iyy="0.00526666666667" iyz="0" izz="0" />
-		</inertial>
-		<collision name="link_left_wheel_collision">
-			<origin rpy="0 1.5707 1.5707" xyz="0 0 0" />
-			<geometry>
-				<cylinder length="0.04" radius="0.1" />
-			</geometry>
-		</collision>
-		<visual name="link_left_wheel_visual">
-			<origin rpy="0 1.5707 1.5707" xyz="0 0 0" />
-			<geometry>
-				<cylinder length="0.04" radius="0.1" />
-			</geometry>
-		</visual>
-	</link>
-	<joint name="joint_right_wheel" type="continuous">
-		<origin rpy="0 0 0" xyz="-0.05 0.15 0"/>
-		<child link="link_right_wheel"/>
-		<parent link="link_chassis" />
-		<axis rpy="0 0 0" xyz="0 1 0"/>
-		<limit effort="10000" velocity="1000"/>
-		<joint_properties damping="1.0" friction="1.0"/>
-	</joint>
-	<joint name="joint_left_wheel" type="continuous">
-		<origin rpy="0 0 0" xyz="-0.05 -0.15 0"/>
-		<child link="link_left_wheel"/>
-		<parent link="link_chassis" />
-		<axis rpy="0 0 0" xyz="0 1 0"/>
-		<limit effort="10000" velocity="1000"/>
-		<joint_properties damping="1.0" friction="1.0"/>
-	</joint>
+	<xacro:link_wheel name="link_right_wheel" />
+	<xacro:joint_wheel name="joint_right_wheel" child="link_right_wheel" origin_xyz="-0.05 0.15 0" />
+	<xacro:link_wheel name="link_left_wheel" />
+	<xacro:joint_wheel name="joint_left_wheel" child="link_left_wheel" origin_xyz="-0.05 -0.15 0" />
 </robot>

Commit message: Add files via upload

File: m2wr_ws/src/m2wr_description/urdf/m2wr.xacro (robot description, xacro)
@@ -46,4 +46,29 @@
 		</visual>
 	</link>
+	<link name="sensor_laser">
+		<inertial>
+			<origin rpy="0 0 0" xyz="0 0 0"/>
+			<mass value="1"/>
+			<xacro:cylinder_inertia mass="1" r="0.05" l="0.1"/>
+		</inertial>
+		<visual>
+			<origin xyz="0 0 0" rpy="0 0 0"/>
+			<geometry>
+				<cylinder radius="0.05" length="0.1" />
+			</geometry>
+			<material name="white" />
+		</visual>
+		<collision>
+			<origin xyz="0 0 0" rpy="0 0 0"/>
+			<geometry>
+				<cylinder radius="0.05" length="0.1"/>
+			</geometry>
+		</collision>
+	</link>
+	<joint name="joint_sensor_laser" type="fixed">
+		<origin xyz="0.15 0 0.05" rpy="0 0 0 "/>
+		<parent link="link_chassis"/>
+		<child link="sensor_laser"/>
+	</joint>
 	<xacro:link_wheel name="link_right_wheel" />
 	<xacro:joint_wheel name="joint_right_wheel" child="link_right_wheel" origin_xyz="-0.05 0.15 0" />

File: m2wr_ws/src/m2wr_description/urdf/macros.xacro (robot description, xacro)
@@ -32,3 +32,9 @@
 		</joint>
 	</macro>
+	<macro name="cylinder_inertia" params="mass l r">
+		<inertia ixx="${mass*(3*r*r+l*l)/12}" ixy="0" ixz="0"
+			iyy="${mass*(3*r*r+l*l)/12}" iyz="0"
+			izz="${mass*(r*r)/2}">
+		</inertia>
+	</macro>
 </robot>

Commit message: Add files via upload

File: m2wr_ws/src/m2wr_description/urdf/m2wr.xacro (robot description, xacro)
@@ -1,77 +1,83 @@
 <?xml version="1.0" ?>
-<robot name="m2wr" xmlns:xacro="http://www.ros.org/wiki/xacro">
-	<xacro:include filename="$(find m2wr_description)/urdf/materials.xacro" />
-	<xacro:include filename="$(find m2wr_description)/urdf/m2wr.gazebo" />
-	<xacro:include filename="$(find m2wr_description)/urdf/macros.xacro" />
-	<link name="link_chassis">
-		<pose>0 0 0.1 0 0 0</pose>
-		<inertial>
-			<mass value="5"/>
-			<origin rpy="0 0 0" xyz="0 0 0.1"/>
-			<inertia ixx="0.0395416666667" ixy="0" ixz="0" iyy="0.106208333333" iyz="0" izz="0"/>
-		</inertial>
-		<collision name="collision_chassis">
-			<geometry>
-				<box size="0.5 0.3 0.07"/>
-			</geometry>
-		</collision>
-		<visual>
-			<origin rpy="0 0 0" xyz="0 0 0"/>
-			<geometry>
-				<box size="0.5 0.3 0.07"/>
-			</geometry>
-			<material name="blue"/>
-		</visual>
-		<collision name="castor_front_collision">
-			<origin rpy="0 0 0" xyz="0.35 0 -0.05" />
-			<geometry>
-				<sphere radius="0.05" />
-			</geometry>
-			<surface>
-				<friction>
-					<ode>
-						<mu>0</mu>
-						<mu2>0</mu2>
-						<slip1>1.0</slip1>
-						<slip2>1.0</slip2>
-					</ode>
-				</friction>
-			</surface>
-		</collision>
-		<visual name="castor_front_visual">
-			<origin rpy="0 0 0" xyz="0.2 0 -0.05" />
-			<geometry>
-				<sphere radius="0.05" />
-			</geometry>
-		</visual>
-	</link>
-	<link name="sensor_laser">
-		<inertial>
-			<origin rpy="0 0 0" xyz="0 0 0"/>
-			<mass value="1"/>
-			<xacro:cylinder_inertia mass="1" r="0.05" l="0.1"/>
-		</inertial>
-		<visual>
-			<origin xyz="0 0 0" rpy="0 0 0"/>
-			<geometry>
-				<cylinder radius="0.05" length="0.1" />
-			</geometry>
-			<material name="white" />
-		</visual>
-		<collision>
-			<origin xyz="0 0 0" rpy="0 0 0"/>
-			<geometry>
-				<cylinder radius="0.05" length="0.1"/>
-			</geometry>
-		</collision>
-	</link>
-	<joint name="joint_sensor_laser" type="fixed">
-		<origin xyz="0.15 0 0.05" rpy="0 0 0 "/>
-		<parent link="link_chassis"/>
-		<child link="sensor_laser"/>
-	</joint>
-	<xacro:link_wheel name="link_right_wheel" />
-	<xacro:joint_wheel name="joint_right_wheel" child="link_right_wheel" origin_xyz="-0.05 0.15 0" />
-	<xacro:link_wheel name="link_left_wheel" />
-	<xacro:joint_wheel name="joint_left_wheel" child="link_left_wheel" origin_xyz="-0.05 -0.15 0" />
+<robot name="m2wr" xmlns:xacro="https://www.ros.org/wiki/xacro" >
+  <!-- include the xacro files-->
+  <xacro:include filename="$(find m2wr_description)/urdf/materials.xacro" />
+  <xacro:include filename="$(find m2wr_description)/urdf/m2wr.gazebo" />
+  <xacro:include filename="$(find m2wr_description)/urdf/macros.xacro" />
+  <!-- Chasis defined here -->
+  <link name="link_chassis">
+    <pose>0 0 0.1 0 0 0</pose>
+    <inertial>
+      <mass value="5"/>
+      <origin rpy="0 0 0" xyz="0 0 0.1"/>
+      <inertia ixx="0.0395416666667" ixy="0" ixz="0" iyy="0.106208333333" iyz="0" izz="0.106208333333"/>
+    </inertial>
+    <collision name="collision_chassis">
+      <geometry>
+        <box size="0.5 0.3 0.07"/>
+      </geometry>
+    </collision>
+    <visual>
+      <origin rpy="0 0 0" xyz="0 0 0"/>
+      <geometry>
+        <box size="0.5 0.3 0.07"/>
+      </geometry>
+      <material name="blue"/>
+    </visual>
+    <!-- caster front -->
+    <collision name="caster_front_collision">
+      <origin rpy=" 0 0 0" xyz="0.35 0 -0.05"/>
+      <geometry>
+        <sphere radius="0.05"/>
+      </geometry>
+      <surface>
+        <friction>
+          <ode>
+            <mu>0</mu>
+            <mu2>0</mu2>
+            <slip1>1.0</slip1>
+            <slip2>1.0</slip2>
+          </ode>
+        </friction>
+      </surface>
+    </collision>
+    <visual name="caster_front_visual">
+      <origin rpy=" 0 0 0" xyz="0.2 0 -0.05"/>
+      <geometry>
+        <sphere radius="0.05"/>
+      </geometry>
+    </visual>
+  </link>
+   <link name="sensor_laser">
+    <inertial>
+      <origin xyz="0 0 0" rpy="0 0 0" />
+      <mass value="1" />
+      <!-- RANDOM INERTIA BELOW -->
+      <xacro:cylinder_inertia mass="1" r="0.05" l="0.1" />
+    </inertial>
+    <visual>
+      <origin xyz="0 0 0" rpy="0 0 0" />
+      <geometry>
+        <cylinder radius="0.05" length="0.1"/>
+      </geometry>
+      <material name="white" />
+    </visual>
+    <collision>
+      <origin xyz="0 0 0" rpy="0 0 0"/>
+      <geometry>
+        <cylinder radius="0.05" length="0.1"/>
+      </geometry>
+    </collision>
+  </link>
+  <joint name="joint_sensor_laser" type="fixed">
+    <origin xyz="0.15 0 0.05" rpy="0 0 0"/>
+    <parent link="link_chassis"/>
+    <child link="sensor_laser"/>
+  </joint>
+  <!-- Create wheel right -->
+   <xacro:link_wheel name="link_right_wheel" />
+   <xacro:joint_wheel name="joint_right_wheel"  child="link_right_wheel"  origin_xyz="-0.05 0.15 0"  />
+  <!-- Left Wheel link -->
+  <xacro:link_wheel name="link_left_wheel" />
+  <xacro:joint_wheel name="joint_left_wheel"   child="link_left_wheel"   origin_xyz="-0.05 -0.15 0"  />
 </robot>

File: m2wr_ws/src/m2wr_description/urdf/macros.xacro (robot description, xacro)
@@ -1,40 +1,38 @@
 <?xml version="1.0"?>
-<robot>
-	<macro name="link_wheel" params="name">
-		<link name="${name}">
-			<inertial>
-				<mass value="0.2" />
-				<origin rpy="0 1.5707 1.5707" xyz="0 0 0" />
-				<inertia ixx="0.00052666666667" ixy="0" ixz="0" iyy="0.00526666666667" iyz="0" izz="0" />
-			</inertial>
-			<collision name="${name}_collision">
-				<origin rpy="0 1.5707 1.5707" xyz="0 0 0" />
-				<geometry>
-				<cylinder length="0.04" radius="0.1" />
-				</geometry>
-			</collision>
-			<visual name="${name}_visual">
-				<origin rpy="0 1.5707 1.5707" xyz="0 0 0" />
-				<geometry>
-					<cylinder length="0.04" radius="0.1" />
-				</geometry>
-			</visual>
-		</link>
-	</macro>
-	<macro name="joint_wheel" params="name child origin_xyz">
-		<joint name="${name}" type="continuous">
-			<origin rpy="0 0 0" xyz="${origin_xyz}"/>
-			<child link="${child}"/>
-			<parent link="link_chassis" />
-			<axis rpy="0 0 0" xyz="0 1 0"/>
-			<limit effort="10000" velocity="1000"/>
-			<joint_properties damping="1.0" friction="1.0"/>
-		</joint>
-	</macro>
-	<macro name="cylinder_inertia" params="mass l r">
-		<inertia ixx="${mass*(3*r*r+l*l)/12}" ixy="0" ixz="0"
-			iyy="${mass*(3*r*r+l*l)/12}" iyz="0"
-			izz="${mass*(r*r)/2}">
-		</inertia>
-	</macro>
+<robot xmlns:xacro="http://www.ros.org/wiki/xacro">
+    <xacro:macro name="link_wheel" params="name">
+        <link name="${name}">
+            <inertial>
+              <mass value="0.2"/>
+              <origin rpy="0 1.5707 1.5707" xyz="0 0 0"/>
+              <inertia ixx="0.000526666666667" ixy="0" ixz="0" iyy="0.000526666666667" iyz="0" izz="0.001"/>
+            </inertial>
+            <collision name="link_right_wheel_collision">
+              <origin rpy="0 1.5707 1.5707" xyz="0 0 0"/>
+              <geometry>
+                <cylinder length="0.04" radius="0.1"/>
+              </geometry>
+            </collision>
+            <visual name="${name}_visual">
+              <origin rpy="0 1.5707 1.5707" xyz="0 0 0"/>
+              <geometry>
+                <cylinder length="0.04" radius="0.1"/>
+              </geometry>
+            </visual>
+        </link>
+    </xacro:macro>
+    <xacro:macro name="joint_wheel" params="name child origin_xyz">
+      <joint name="${name}" type="continuous">
+        <origin rpy="0 0 0" xyz="${origin_xyz}"/>
+        <child link="${child}"/>
+        <parent link="link_chassis"/>
+        <axis rpy="0 0 0" xyz="0 1 0"/>
+        <limit effort="10000" velocity="1000"/>
+        <joint_properties damping="1.0" friction="1.0"/>
+      </joint>
+    </xacro:macro>
+    <xacro:macro name="cylinder_inertia" params="mass r l">
+      <inertia ixx="${mass*(3*r*r+l*l)/12}" ixy = "0" ixz = "0"
+                iyy="${mass*(3*r*r+l*l)/12}" iyz = "0" izz="${mass*(r*r)/2}" />
+    </xacro:macro>
 </robot>

File: m2wr_ws/src/m2wr_description/urdf/materials.xacro (robot description, xacro)
@@ -1,24 +1,27 @@
-<?xml version="1.0"?>
-<robot>
-	<material name="black">
-		<color rgba="0.0 0.0 0.0 1.0"/>
-	</material>
-	<material name="blue">
-		<color rgba="0.203125 0.238281250 0.285156250 1.0"/>
-	</material>
-	<material name="green">
-		<color rgba="0.0 0.8 0.0 1.0"/>
-	</material>
-	<material name="grey">
-		<color rgba="0.2 0.2 0.2 1.0"/>
-	</material>
-	<material name="orange">
-		<color rgba="1.0 0.4235294117650 0.0392156862745 1.0"/>
-	</material>
-	<material name="brown">
-		<color rgba="0.870588235294 0.8117647058820 0.7647058823530 1.0"/>
-	</material>
-	<material name="white">
-		<color rgba="1.0 1.0 1.0 1.0"/>
-	</material>
+<?xml version="1.0" ?>
+<robot name="m2wr" xmlns:xacro="https://www.ros.org/wiki/xacro" >
+  <material name="black">
+    <color rgba="0.0 0.0 0.0 1.0"/>
+  </material>
+  <material name="blue">
+    <color rgba="0.203125 0.23828125 0.28515625 1.0"/>
+  </material>
+  <material name="green">
+    <color rgba="0.0 0.8 0.0 1.0"/>
+  </material>
+  <material name="grey">
+    <color rgba="0.2 0.2 0.2 1.0"/>
+  </material>
+  <material name="orange">
+    <color rgba="1.0 0.423529411765 0.0392156862745 1.0"/>
+  </material>
+  <material name="brown">
+    <color rgba="0.870588235294 0.811764705882 0.764705882353 1.0"/>
+  </material>
+  <material name="red">
+    <color rgba="0.80078125 0.12890625 0.1328125 1.0"/>
+  </material>
+  <material name="white">
+    <color rgba="1.0 1.0 1.0 1.0"/>
+  </material>
 </robot>
